Commit message: chore: removed unused dockerfiles

File: ros2/teachingless/assets/ur_description/urdf/ur5e.urdf (robot description, URDF)
Before this commit: robot ur, 13 links, 12 joints
Links:
- link base_link_inertia: geometry collision mesh filename=../meshes/ur5e/collision/base.stl; visual mesh filename=../meshes/ur5e/visual/base.dae
- link forearm_link: geometry collision mesh filename=../meshes/ur5e/collision/forearm.stl; visual mesh filename=../meshes/ur5e/visual/forearm.dae
- link shoulder_link: geometry collision mesh filename=../meshes/ur5e/collision/shoulder.stl; visual mesh filename=../meshes/ur5e/visual/shoulder.dae
- link upper_arm_link: geometry collision mesh filename=../meshes/ur5e/collision/upperarm.stl; visual mesh filename=../meshes/ur5e/visual/upperarm.dae
- link wrist_1_link: geometry collision mesh filename=../meshes/ur5e/collision/wrist1.stl; visual mesh filename=../meshes/ur5e/visual/wrist1.dae
- link wrist_2_link: geometry collision mesh filename=../meshes/ur5e/collision/wrist2.stl; visual mesh filename=../meshes/ur5e/visual/wrist2.dae
- link wrist_3_link: geometry collision mesh filename=../meshes/ur5e/collision/wrist3.stl; visual mesh filename=../meshes/ur5e/visual/wrist3.dae
